Commit message: Update Stability Check and Block Size

File: DATA/block.urdf (robot description, URDF)
Before this commit: robot block_2, 1 links, 0 joints
Links:
- link block_2_base_link: geometry collision box size=0.08 0.04 0.04; visual box size=0.08 0.04 0.04

Commit message: Minor Test Update

File: DATA/block.urdf (robot description, URDF)
Before this commit: robot block_2, 1 links, 0 joints
Links:
- link block_2_base_link: mass 0.02 -> 0.3072
