Commit message: Update to Compas_client, Update block size, Update Gofa model

File: assembly_gymenv/DATA/block.urdf (robot description, URDF)
Before this commit: robot block_2, 1 links, 0 joints
Links:
- link block_2_base_link: mass 0.3072 -> 0.25; geometry collision box size=0.10 0.05 0.05; visual box size=0.10 0.05 0.05
